File: hardware/openkey-cps1.kicad_sch (KiCad schematic)
At the start: 17 parts, among them J1 CND Top, J2 CNC Top, J3 CNA Top, J4 CNB Top, J5 CND Bottom, J6 CNC Bottom, J7 CNA Bottom, J8 CNB Bottom, J9 Conn_01x03_Female, SW1 SW_DIP_x05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

Commit message: Updated hardware/firmware that adds an optional reset header
The optional reset header that can be used to hookup openkey-cps1
to the A board's reset signal to allow openkey to control it.  In
general you shouldn't need this, but waited to make it an available
option.  More details are in the README.md

The updated firmware is backwards compatible with the previous
hardware revision.
Parts:
- added J11: Conn_01x03_Pin, openkey:PinHeader_1x03_P2.54mm_Vertical, symbol Connector:Conn_01x03_Pin
- C1: footprint openkey-cps1:C_0805_2012Metric_Pad1.18x1.45mm_HandSolder_alt -> openkey:C_0805_2012Metric_Pad1.18x1.45mm_HandSolder
Connections:
- net GND: now also J11.2 (Pin_2)
- net RESET: now reaches U1.13 (PA3)
- net RESET: now also J11.1 (Pin_1)
- net RESET_DELAY: now reaches U1.7 (PB2)
- net RESET_DELAY: now also J11.3 (Pin_3)
- no-connect marks 4 -> 2
Other:
- note added: "Reset Header"
